File: AuxPSU.kicad_sch (KiCad schematic)
At the start: 10 parts, among them U4 TPS5430DDA

Commit message: Make ERC happy
Changed lines of the file:
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@@
 (kicad_sch
-	(version 20231120)
+	(version 20250114)
 	(generator "eeschema")
-	(generator_version "8.0")
+	(generator_version "9.0")
 	(paper "A3")
 	(junction
@@
 		(shape input)
 		(at 146.05 133.35 180)
-		(fields_autoplaced yes)
 		(effects
 			(font
@@
 		(shape input)
 		(at 111.76 123.19 180)
-		(fields_autoplaced yes)
 		(effects
 			(font
@@
 		(shape output)
 		(at 278.13 123.19 0)
-		(fields_autoplaced yes)
 		(effects
 			(font

Commit message: Switch R0402 to 0603
Parts:
- R46: footprint Resistor_SMD:R_0402_1005Metric -> Resistor_SMD:R_0603_1608Metric; JLC C25744 -> C25804
Changed lines of the file:
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@@
 			)
 		)
-		(property "Footprint" "Resistor_SMD:R_0402_1005Metric"
+		(property "Footprint" "Resistor_SMD:R_0603_1608Metric"
 			(at 151.638 137.16 90)
 			(effects
@@
 			)
 		)
-		(property "JLC" "C25744"
+		(property "JLC" "C25804"
 			(at 149.86 137.16 0)
 			(effects

Commit message: Fix BOM and parts placement
Parts:
- C13: FT Rotation Offset (none) -> 180
Changed lines of the file:
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@@
 			)
 		)
-		(property "APPLICATION" ""
+		(property "FT Rotation Offset" "180"
 			(at 259.08 128.27 0)
 			(effects
