File: Core.kicad_sch (KiCad schematic)
At the start: 5 parts, among them J25 Conn_01x05_Pin, J26 xcore, U7 M24C02-WMN

Commit message: EEPROM header now DNP (Fixes #16)
Parts:
- J25: now not fitted
Changed lines of the file:
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@@
 		(in_bom yes)
 		(on_board yes)
-		(dnp no)
+		(dnp yes)
 		(fields_autoplaced yes)
 		(property "Reference" "J25"
