File: Connectors.kicad_sch (KiCad schematic)
At the start: 20 parts, among them J16 USB_A_Stacked, J22 HR911130A, J23 HR911130A, J24 HR911130A, U1 TPS2065CDBV

Commit message: Fixed resistor values, small changes
Other:
- note added: "DNP this connector, otherwise the YardForce Classic 500 won't close without modifying the top half of the robot"
- note added: "USB 2 Power Switches and Connectors Power is always on, switches are there for safety (they will deliver max 1A and shut off on overcurrent)"
- note removed: "USB 2 Power Switches and Connectors Power is always on, switches are there for safety (they will deliver max 1A)"
- moved on the sheet: C1, C21, C22, C23, C3, C4, C5, J16, J22, J23, J24, R1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

Commit message: Add USB 3D via nlbn
Parts:
- J16: footprint Connector_USB:USB_A_Wuerth_61400826021_Horizontal_Stacked -> nlbn:USB-269-BRW_C720548_MOD
Changed lines of the file:
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@@
 			)
 		)
-		(property "Footprint" "Connector_USB:USB_A_Wuerth_61400826021_Horizontal_Stacked"
+		(property "Footprint" "nlbn:USB-269-BRW_C720548_MOD"
 			(at 71.12 201.93 0)
 			(effects

Commit message: Add Robot-Adapter and OEM plugs WIP
Parts:
- C21, J23, R10, R9: now not fitted
Changed lines of the file:
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@@
 	(wire
 		(pts
-			(xy 234.95 81.28) (xy 234.95 96.52)
+			(xy 234.95 81.28) (xy 234.95 87.63)
 		)
 		(stroke
@@
 		(in_bom yes)
 		(on_board yes)
-		(dnp no)
+		(dnp yes)
 		(fields_autoplaced yes)
 		(property "Reference" "J23"
@@
 	(symbol
 		(lib_id "power:GND")
-		(at 234.95 96.52 0)
+		(at 234.95 87.63 0)
 		(unit 1)
 		(exclude_from_sim no)
@@
 		(fields_autoplaced yes)
 		(property "Reference" "#PWR035"
-			(at 234.95 102.87 0)
+			(at 234.95 93.98 0)
 			(effects
 				(font
@@
 		)
 		(property "Value" "GND"
-			(at 234.95 101.6 0)
+			(at 234.95 92.71 0)
 			(effects
 				(font
@@
 		)
 		(property "Footprint" ""
-			(at 234.95 96.52 0)
+			(at 234.95 87.63 0)
 			(effects
 				(font
@@
 		)
 		(property "Datasheet" ""
-			(at 234.95 96.52 0)
+			(at 234.95 87.63 0)
 			(effects
 				(font
@@
 		)
 		(property "Description" "Power symbol creates a global label with name \"GND\" , ground"
-			(at 234.95 96.52 0)
+			(at 234.95 87.63 0)
 			(effects
 				(font
@@
 		(exclude_from_sim no)
 		(in_bom yes)
-		(on_board yes)
+		(on_board no)
 		(dnp yes)
 		(fields_autoplaced yes)
@@
 		(exclude_from_sim no)
 		(in_bom yes)
-		(on_board yes)
-		(dnp no)
+		(on_board no)
+		(dnp yes)
 		(fields_autoplaced yes)
 		(property "Reference" "R9"
@@
 		(exclude_from_sim no)
 		(in_bom yes)
-		(on_board yes)
-		(dnp no)
+		(on_board no)
+		(dnp yes)
 		(fields_autoplaced yes)
 		(property "Reference" "C21"
@@
 		(exclude_from_sim no)
 		(in_bom yes)
-		(on_board yes)
-		(dnp no)
+		(on_board no)
+		(dnp yes)
 		(fields_autoplaced yes)
 		(property "Reference" "R10"

Commit message: Fix BOM and switch C0402 to C0603
Parts:
- C1, C22, C23, C5: footprint Capacitor_SMD:C_0402_1005Metric -> Capacitor_SMD:C_0603_1608Metric; JLC C307331 -> C14663
Changed lines of the file:
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@@
 			)
 		)
-		(property "Footprint" "Capacitor_SMD:C_0402_1005Metric"
+		(property "Footprint" "Capacitor_SMD:C_0603_1608Metric"
 			(at 95.25 167.3352 0)
 			(effects
@@
 			)
 		)
-		(property "JLC" "C307331"
+		(property "JLC" "C14663"
 			(at 99.06 166.37 0)
 			(effects
@@
 			)
 		)
-		(property "Footprint" "Capacitor_SMD:C_0402_1005Metric"
+		(property "Footprint" "Capacitor_SMD:C_0603_1608Metric"
 			(at 53.34 140.6652 0)
 			(effects
@@
 			)
 		)
-		(property "JLC" "C307331"
+		(property "JLC" "C14663"
 			(at 57.15 139.7 0)
 			(effects
@@
 			)
 		)
-		(property "Footprint" "Capacitor_SMD:C_0402_1005Metric"
+		(property "Footprint" "Capacitor_SMD:C_0603_1608Metric"
 			(at 234.95 198.4248 0)
 			(effects
@@
 			)
 		)
-		(property "JLC" "C307331"
+		(property "JLC" "C14663"
 			(at 231.14 199.39 0)
 			(effects
@@
 			)
 		)
-		(property "Footprint" "Capacitor_SMD:C_0402_1005Metric"
+		(property "Footprint" "Capacitor_SMD:C_0603_1608Metric"
 			(at 234.95 110.7948 0)
 			(effects
@@
 			)
 		)
-		(property "JLC" "C307331"
+		(property "JLC" "C14663"
 			(at 231.14 111.76 0)
 			(effects

Commit message: Switch R0402 to 0603
Parts:
- R1, R3: footprint Resistor_SMD:R_0402_1005Metric -> Resistor_SMD:R_0603_1608Metric; JLC C25744 -> C25804
Changed lines of the file:
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@@
 			)
 		)
-		(property "Footprint" "Resistor_SMD:R_0402_1005Metric"
+		(property "Footprint" "Resistor_SMD:R_0603_1608Metric"
 			(at 58.42 146.558 90)
 			(effects
@@
 			)
 		)
-		(property "JLC" "C25744"
+		(property "JLC" "C25804"
 			(at 58.42 144.78 0)
 			(effects
@@
 			)
 		)
-		(property "Footprint" "Resistor_SMD:R_0402_1005Metric"
+		(property "Footprint" "Resistor_SMD:R_0603_1608Metric"
 			(at 76.2 126.492 90)
 			(effects
@@
 			)
 		)
-		(property "JLC" "C25744"
+		(property "JLC" "C25804"
 			(at 76.2 128.27 0)
 			(effects

Commit message: Final part rotations
Parts:
- U1: FT Rotation Offset (none) -> 90
Changed lines of the file:
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@@
 			)
 		)
-		(property "APPLICATION" ""
+		(property "FT Rotation Offset" "90"
 			(at 76.2 142.24 0)
 			(effects
